File: DRV, Coupler, PA.kicad_sch (KiCad schematic)
At the start: 70 parts, among them K1 G6K-2P-Y(80, 60m), K2 G6K-2P-Y(40, 30m), K3 G6K-2P-Y(20, 17, 15m), K4 G6K-2P-Y(12, 11, 10m), Q1 BD139, Q2 IRFP250, Q3 IRFP250, Q4 BD139

Commit message: Driver done.
Parts:
- removed C23: 10uF, symbol Device:C_Polarized_Small
- removed C25: 100nF, symbol Device:C_Small
- removed L4: RFC 10uH/100 mA, symbol Device:L_Ferrite_Small
- removed R11: 4k7, symbol Device:R_Small
- removed RV3: 1k - Bias 2, symbol Device:R_Potentiometer_Trim
- added C18, C20, C23, C34, C37: 100nF, symbol Device:C_Small
- added C19, C24, C25, C35: 10uF, symbol Device:C_Polarized_Small
- added C21: 68nF, symbol Device:C_Small
- added D9: 1N4148, Diode_THT:D_DO-35_SOD27_P7.62mm_Horizontal, symbol Diode:1N4148
- added L1: DRV_In, symbol Intralha.:L_Ferrite_Taped_Coupled_Small
- added L14: RFC 10uH/100 mA, symbol Device:L_Ferrite_Small
- added L2, L3: RFC 10uH/5A, symbol Device:L_Ferrite_Small
- added L4: DRV_Out, symbol Intralha.:L_Ferrite_Taped_Coupled_Small
- added Q3, Q4: BD139, Package_TO_SOT_THT:TO-126-3_Vertical, symbol Transistor_BJT:BD139
- added R20, R5: 1k, symbol Device:R_Small
- added R22: 4k7, symbol Device:R_Small
- added R33, R34: 74k, symbol Device:R_Small
- added R6, R7: 60R/No ind, symbol Device:R_Small
- added R8: 0.35R/No ind, symbol Device:R_Small
- added RV2: 10k, symbol Device:R_Potentiometer_Trim
- added RV4: 1k - Bias 1, symbol Device:R_Potentiometer_Trim
- C22: value 100nF -> 68nF
- R9: value 1k -> 0.35R/No ind
- RV1: value 10k -> 2k
- renumbered C18 to C26, C19 to C27, C20 to C28, C21 to C29, C35 to C30, C36 to C31, C37 to C32, C38 to C33, C24 to C36, C26 to C38, C27 to C39, C28 to C40, C29 to C41, C30 to C42, C31 to C43, C32 to C44, C33 to C45, C34 to C46, D9 to D10, D10 to D11, L3 to L13, L5 to L15, L6 to L16, L1 to L5, L2 to L6, Q4 to Q2, Q2 to Q5, Q3 to Q6, R5 to R10, R6 to R11, R7 to R12, R8 to R13, R22 to R14, R23 to R15, R24 to R16, R25 to R17, R26 to R18, R27 to R19, R10 to R21, R12 to R23, R13 to R24, R14 to R25, R15 to R26, R16 to R27, R17 to R28, R18 to R29, R19 to R30, R20 to R31, R21 to R32, RV2 to RV3
Connections:
- net +12V_SW: now also K1.1, K2.1, K3.1, K4.1, L2.2, L3.2, Q4.2 (C), R20.1, R5.1; no longer R9.1
- net GND: now also RV3.1, C18.1, C19.2, C20.1, C23.1, C24.2, C25.2, C34.1, C35.2, C37.1, RV2.1, RV4.1; no longer C22.1, D8.2 (A), RV1.2
- net at C36.2, L13.1, RV3.2: no longer RV3.1
- net at Q2.1 (E): now also R8.2
- net at Q2.2 (C): now also C20.2, C24.1, L2.1
- net at Q2.3 (B): now also C21.1, R33.1
- net at D8.1 (K), Q1.3 (B): now also RV1.2; no longer R9.2, RV1.3
- net at R24.2: now also L14.2
- net DRV_IN 1: no longer names the net of C28.2, R10.1
- net DRV_IN 1: now also L4.4
- net DRV_IN 2: no longer names the net of C29.2, R11.1
- net DRV_IN 2: now also L4.3
- new net: Q3.1 (E), R9.2
- new net: C23.2, C25.1, L3.1, Q3.2 (C)
- new net: C22.1, Q3.3 (B), R34.2
- new net: C34.2, C35.1, D9.2 (A), Q4.1 (E), R21.1, R22.1
- new net: R22.2, RV4.3
- new net: R5.2, RV1.3
- new net: L4.2, R8.1
- new net: C18.2, C19.1, D8.2 (A), L4.5 (Tap), Q1.1 (E), R33.2, R34.1
- new net: C37.2, L14.1, RV4.2
- new net: D9.1 (K), Q4.3 (B), RV2.2
- new net: R20.2, RV2.3
- new net: L1.4, R6.1
- new net: C21.2, R6.2
- new net: L1.3, R7.1
- new net: C22.2, R7.2
- new net: L4.1, R9.1
Other:
- moved on the sheet: Q2

Commit message: Driver correction
Parts:
- removed C22: 68nF, symbol Device:C_Small
- removed C23: 100nF, symbol Device:C_Small
- removed C24, C25: 10uF, symbol Device:C_Polarized_Small
- removed L3: RFC 10uH/5A, symbol Device:L_Ferrite_Small
- removed R33, R34: 74k, symbol Device:R_Small
- added C44: 100nF, symbol Device:C_Small
- added L4: RFC 15uH/1A, symbol Device:L_Ferrite_Small
- C20: value 100nF -> 10nF
- C21: value 68nF -> 100nF
- L2: value RFC 10uH/5A -> RFC 30uH/0.5A
- R5: renamed from R6; value 60R/No ind -> 35R/No ind
- R6: renamed from R7; value 60R/No ind -> 35R/No ind
- renumbered C19 to C18, C18 to C19, C26 to C22, C27 to C23, C28 to C24, C29 to C25, C30 to C26, C31 to C27, C32 to C28, C33 to C29, C34 to C30, C35 to C31, C36 to C32, C37 to C33, C38 to C34, C39 to C35, C40 to C36, C41 to C37, C42 to C38, C43 to C39, C44 to C40, C45 to C41, C46 to C42, L4 to L3, R5 to R7
Connections:
- net +12V_SW: now also L4.2; no longer L2.2
- net GND: now also C21.1, R8.1, R9.2, C44.1
- net at Q3.1 (E): now also R9.1; no longer R9.2
- net at Q3.2 (C): now also L3.1
- net at Q3.3 (B): now also R6.2
- net at L3.2: now also Q2.2 (C); no longer R8.1
- net at Q2.3 (B): now also R5.2; no longer C21.1
- net at C18.1, C19.2, D8.2 (A)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: now also L2.2; no longer L3.5 (Tap)
- net at R5.1: now also L1.1; no longer L1.4
- net at C21.2: now also C20.2, L3.5 (Tap), L4.1; no longer R5.2
- net at R6.1: now also L1.2; no longer L1.3
- net at L1.5 (Tap): now also L2.1, C44.2
Other:
- moved on the sheet: C18, C19, D8, L1, Q1, Q2, Q3, R7, RV1

Commit message: Pre-Driver Work
Parts:
- removed L1: DRV_In, symbol Intralha.:L_Ferrite_Taped_Coupled_Small
- added C21, C23: 100nF, symbol Device:C_Small
- added C22: 10uF, symbol Device:C_Polarized_Small
- added C47, C48: 150nF, symbol Device:C_Small
- added D8: 1N4148, Diode_THT:D_DO-35_SOD27_P7.62mm_Horizontal, symbol Diode:1N4148
- added L1: Pre DRV Out/DRV In, symbol Intralha.:L_Ferrite_Taped_Coupled_Small_2
- added L3: RFC 30uH/0.5A, symbol Device:L_Ferrite_Small
- added L5: Pre Drv In, symbol Intralha.:L_Ferrite_Taped_Coupled_Small_2
- added Q1: BD139, Package_TO_SOT_THT:TO-126-3_Vertical, symbol Transistor_BJT:BD139
- added Q3, Q4: 2N3866, Package_TO_SOT_THT:TO-39-3, symbol Transistor_BJT:2N2219
- added R10, R11: 1R/0,5W/No ind, symbol Device:R_Small
- added R38, R39: 35R, symbol Device:R_Small
- added R40, R41: 18R/No ind, symbol Device:R_Small
- added R5: 1k, symbol Device:R_Small
- added R8, R9: 35R/No ind, symbol Device:R_Small
- added RV1: 2k, symbol Device:R_Potentiometer_Trim
- renumbered C44 to C18, C18 to C19, C19 to C20, C20 to C24, C21 to C25, C22 to C26, C23 to C27, C24 to C28, C25 to C29, C26 to C30, C27 to C31, C28 to C32, C29 to C33, C30 to C34, C31 to C35, C32 to C36, C33 to C37, C34 to C38, C35 to C39, C36 to C40, C37 to C41, C38 to C42, C39 to C43, C40 to C44, C41 to C45, C42 to C46, D9 to D10, D10 to D11, D11 to D12, D8 to D9, L8 to L10, L9 to L11, L10 to L12, L11 to L13, L12 to L14, L13 to L15, L14 to L16, L15 to L17, L16 to L18, L3 to L4, L4 to L6, L5 to L7, L6 to L8, L7 to L9, Q1 to Q2, Q2 to Q5, Q3 to Q6, Q4 to Q7, Q5 to Q8, Q6 to Q9, R7 to R12, R8 to R13, R9 to R14, R10 to R15, R11 to R16, R12 to R17, R13 to R18, R14 to R19, R15 to R20, R16 to R21, R17 to R22, R18 to R23, R19 to R24, R20 to R25, R21 to R26, R22 to R27, R23 to R28, R24 to R29, R25 to R30, R26 to R31, R27 to R32, R28 to R33, R29 to R34, R30 to R35, R31 to R36, R32 to R37, R5 to R6, R6 to R7, RV1 to RV2, RV2 to RV3, RV3 to RV4, RV4 to RV5
Connections:
- net +12V_SW: now also Q1.2 (C), R5.1
- net GND: now also C21.1, C22.2, C23.1, C47.1, C48.1, R10.2, R11.2, R38.2, R39.2, RV1.1
- net at C18.2, L2.1: now also L1.5 (Tap)
- net at R6.1: now also L1.4, R40.1
- net at R7.1: now also L1.3, R41.1
- new net: R5.2, RV1.3
- new net: C21.2, C22.1, D8.2 (A), L3.2, Q1.1 (E)
- new net: Q4.1 (E), R11.1
- new net: L1.1, Q4.3 (C)
- new net: L1.2, Q3.3 (C)
- new net: Q3.2 (B), R39.1, R8.1
- new net: L5.3, R8.2
- new net: C23.2, L3.1, L5.5 (Tap)
- new net: D8.1 (K), Q1.3 (B), RV1.2
- new net: Q3.1 (E), R10.1
- new net: C47.2, R41.2
- new net: L5.4, R9.2
- new net: Q4.2 (B), R38.1, R9.1
- new net: C48.2, R40.2
Other:
- moved on the sheet: C18, L2

Commit message: Pre-Driver Work 0.2
Parts:
- R38, R39: value 35R -> 35R/No ind
Other:
- moved on the sheet: L5
Changed lines of the file:
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@@
 	(wire
 		(pts
-			(xy 50.8 171.45) (xy 74.93 171.45)
+			(xy 50.8 171.45) (xy 66.04 171.45)
 		)
 		(stroke
@@
 	(wire
 		(pts
-			(xy 74.93 127) (xy 50.8 127)
+			(xy 66.04 127) (xy 50.8 127)
 		)
 		(stroke
@@
 	(wire
 		(pts
-			(xy 74.93 127) (xy 74.93 134.62)
+			(xy 66.04 127) (xy 66.04 134.62)
 		)
 		(stroke
@@
 	(wire
 		(pts
-			(xy 74.93 171.45) (xy 74.93 139.7)
+			(xy 66.04 171.45) (xy 66.04 139.7)
 		)
 		(stroke
@@
 	(wire
 		(pts
-			(xy 72.39 137.16) (xy 52.07 137.16)
+			(xy 63.5 137.16) (xy 52.07 137.16)
 		)
 		(stroke
@@
 			)
 		)
-		(property "Value" "35R"
+		(property "Value" "35R/No ind"
 			(at 43.18 129.54 0)
 			(effects
@@
 	(symbol
 		(lib_id "Intralha.:L_Ferrite_Taped_Coupled_Small_2")
-		(at 76.2 137.16 270)
+		(at 67.31 137.16 270)
 		(unit 1)
 		(exclude_from_sim no)
@@
 		(fields_autoplaced yes)
 		(property "Reference" "L5"
-			(at 78.74 135.8899 90)
+			(at 69.85 135.8899 90)
 			(effects
 				(font
@@
 		)
 		(property "Value" "Pre Drv In"
-			(at 78.74 138.4299 90)
+			(at 69.85 138.4299 90)
 			(effects
 				(font
@@
 		)
 		(property "Footprint" ""
-			(at 76.2 137.16 0)
+			(at 67.31 137.16 0)
 			(effects
 				(font
@@
 		)
 		(property "Datasheet" ""
-			(at 76.2 137.16 0)
+			(at 67.31 137.16 0)
 			(effects
 				(font
@@
 		)
 		(property "Description" "Ferrite core taped, small symbol"
-			(at 76.2 137.16 0)
+			(at 67.31 137.16 0)
 			(effects
 				(font
@@
 			)
 		)
-		(property "Value" "35R"
-			(at 38.1 173.99 0)
+		(property "Value" "35R/No ind"
+			(at 34.29 173.99 0)
 			(effects
 				(font

Commit message: huge modification of the project.
Parts:
- removed C30: 35pF, symbol Device:C_Trim_Small
- removed C31: 27pF, symbol Device:C_Trim_Small
- removed C32: 17pF, symbol Device:C_Trim_Small
- removed C33: 10pF, symbol Device:C_Trim_Small
- removed C38: 10uF, symbol Device:C_Polarized_Small
- removed C39, C43, C44, C45: 100nF, symbol Device:C_Small
- removed C40, C42: 100pF, symbol Device:C_Small
- removed C41: 10nF, symbol Device:C_Small
- removed C46: 1nF, symbol Device:C_Small
- removed D11, D12: SMBJ15CA, Diode_THT:D_DO-201AE_P15.24mm_Horizontal, symbol Diode:1N62xxCA
- removed K1: G6K-2P-Y(80, 60m), symbol Relay:G6K-2
- removed K2: G6K-2P-Y(40, 30m), symbol Relay:G6K-2
- removed K3: G6K-2P-Y(20, 17, 15m), symbol Relay:G6K-2
- removed K4: G6K-2P-Y(12, 11, 10m), symbol Relay:G6K-2
- removed L10, L9: 1.5uH, symbol Device:L_Small
- removed L11, L12: 680nH, symbol Device:L_Small
- removed L13, L14: 330nH, symbol Device:L_Small
- removed L17: RFC 10uH/15A, symbol Device:L_Ferrite_Small
- removed L18: T_Out, symbol Intralha.:L_Ferrite_Taped_Coupled_Small
- removed L7, L8: 3uH, symbol Device:L_Small
- removed Q8, Q9: IRFP250, symbol Simulation_SPICE:NMOS
- removed R17, R18, R19, R20, R21, R22, R23, R24: 6R8/No ind, symbol Device:R_Small
- removed R28, R29: 6R8(1/4W no ind.), symbol Device:R_Small
- removed R30, R31: 100k no ind., symbol Device:R_Small
- removed R32, R33: 150R(1/4W no ind.), symbol Device:R_Small
- removed R34, R35: 0,1R/3W no ind., symbol Device:R_Small
- removed R36, R37: 100k, symbol Device:R_Small
- renumbered C47 to C26, C48 to C27, C18 to C28, C19 to C29, C20 to C30, C21 to C31, C22 to C32, C23 to C33, C24 to C34, C25 to C35, C26 to C36, C27 to C37, C28 to C38, C29 to C39, C34 to C40, C35 to C41, C36 to C42, C37 to C43, D8 to D10, D9 to D11, D10 to D12, L15 to L7, L16 to L8, R39 to R10, R38 to R11, R8 to R12, R9 to R13, R10 to R14, R11 to R15, R12 to R16, R13 to R17, R14 to R18, R15 to R19, R16 to R20, R25 to R21, R26 to R22, R27 to R23, R41 to R5, R40 to R6, R5 to R7, R6 to R8, R7 to R9
Other:
- note removed: "BUS_DRV_1"
- note removed: "BUS_DRV_2"
- note removed: "BUS_GATE_1"
- note removed: "BUS_GATE_2"
- moved on the sheet: C40, C41, C42, C43, D12, L7, L8, Q7, R21, R22, R23, RV3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
