File: control.kicad_sch (KiCad schematic)
At the start: 4 parts, among them SW3 Reset, U4 ULN2803A

Commit message: Logical Work
Parts:
- renumbered A2 to A1, C64 to C1, SW3 to SW1, U4 to U1
Changed lines of the file:
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@@
 		(dnp no)
 		(fields_autoplaced yes)
-		(property "Reference" "#PWR0103"
+		(property "Reference" "#PWR01"
 			(at 91.44 88.9 0)
 			(effects
@@
 			(project "Omega Radio"
 				(path "/3468ce30-82a7-4087-a7ac-02063723d842/054ac589-6dd1-4df0-b655-78f47df0dd4e"
-					(reference "#PWR0103")
+					(reference "#PWR01")
 					(unit 1)
 				)
@@
 		(on_board yes)
 		(dnp no)
-		(property "Reference" "C64"
+		(property "Reference" "C1"
 			(at 94.488 81.026 0)
 			(do_not_autoplace yes)
@@
 			(project "Omega Radio"
 				(path "/3468ce30-82a7-4087-a7ac-02063723d842/054ac589-6dd1-4df0-b655-78f47df0dd4e"
-					(reference "C64")
+					(reference "C1")
 					(unit 1)
 				)
@@
 		(dnp no)
 		(fields_autoplaced yes)
-		(property "Reference" "#PWR0104"
+		(property "Reference" "#PWR02"
 			(at 130.81 170.18 0)
 			(effects
@@
 			(project "Omega Radio"
 				(path "/3468ce30-82a7-4087-a7ac-02063723d842/054ac589-6dd1-4df0-b655-78f47df0dd4e"
-					(reference "#PWR0104")
+					(reference "#PWR02")
 					(unit 1)
 				)
@@
 		(dnp no)
 		(fields_autoplaced yes)
-		(property "Reference" "U4"
+		(property "Reference" "U1"
 			(at 130.81 130.81 0)
 			(effects
@@
 			(project "Omega Radio"
 				(path "/3468ce30-82a7-4087-a7ac-02063723d842/054ac589-6dd1-4df0-b655-78f47df0dd4e"
-					(reference "U4")
+					(reference "U1")
 					(unit 1)
 				)
@@
 		(on_board yes)
 		(dnp no)
-		(property "Reference" "SW3"
+		(property "Reference" "SW1"
 			(at 89.408 73.66 90)
 			(effects
@@
 			(project "Omega Radio"
 				(path "/3468ce30-82a7-4087-a7ac-02063723d842/054ac589-6dd1-4df0-b655-78f47df0dd4e"
-					(reference "SW3")
+					(reference "SW1")
 					(unit 1)
 				)
@@
 		(on_board yes)
 		(dnp no)
-		(property "Reference" "A2"
+		(property "Reference" "A1"
 			(at 127 80.01 0)
 			(effects
@@
 			(project "Omega Radio"
 				(path "/3468ce30-82a7-4087-a7ac-02063723d842/054ac589-6dd1-4df0-b655-78f47df0dd4e"
-					(reference "A2")
+					(reference "A1")
 					(unit 1)
 				)
