File: DRV, PA.kicad_sch (KiCad schematic)
At the start: 26 parts, among them Q1 2SC5171, Q2 2SA1930, Q3 IRF630, Q4 IRF630

Commit message: Bias Work
Parts:
- removed L2: PA_Out, symbol Intralha.:L_Ferrite_Taped_Coupled_Small_2
- added C29, C31, C32: 100nF, symbol Device:C_Small
- added C30: 10uF, symbol Device:C_Polarized_Small
- added C33, C34: 84pF, symbol Device:C_Small
- added D12: 1N4148, Diode_THT:D_DO-35_SOD27_P7.62mm_Horizontal, symbol Diode:1N4148
- added L5: PA_Out, symbol Intralha.:L_Ferrite_Taped_Coupled_Small_2
- added L6, L7: 10uH/100mA, symbol Device:L_Ferrite_Small
- added Q5: BD139, Package_TO_SOT_THT:TO-126-3_Vertical, symbol Transistor_BJT:BD139
- added R12: 18k, symbol Device:R_Small
- added R13, R14: 4k7, symbol Device:R_Small
- added R15, R18: 125R/No ind, symbol Device:R_Small
- added R16, R17: 100k/No ind, symbol Device:R_Small
- added RV1: 10k, symbol Device:R_Potentiometer_Trim
- added RV2: 10k - Bias 1, symbol Device:R_Potentiometer_Trim
- added RV3: 10k - Bias 2, symbol Device:R_Potentiometer_Trim
- renumbered C17 to C21, C19 to C22, C18 to C23, C20 to C24, C15 to C25, C21 to C26, C16 to C27, C22 to C28, D7 to D10, D8 to D11, D9 to D8, D10 to D9
Connections:
- net +24V_Main: now also Q5.2 (C), R12.1
- net GND: now also C29.1, C30.2, C31.1, C32.1, C33.1, C34.2, R16.1, R17.1, RV1.1, RV2.1, RV3.1
- net at R7.2, R8.1, R9.1: now also L6.2, L7.2
- net at D11.1 (K), Q4.1 (G), R11.2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: now also R17.2, R18.1
- net at Q3.2 (D), Q4.2 (D): now also L5.2
- net at D10.1 (K), Q3.1 (G), R10.2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: now also R15.1, R16.2
- net at C26.1, C28.1, L4.2: now also L5.3 (Tap)
- new net: C33.2, R15.2
- new net: C29.2, C30.1, D12.2 (A), Q5.1 (E), R13.1, R14.1
- new net: R14.2, RV3.3
- new net: C31.2, L6.1, RV2.2
- new net: C32.2, L7.1, RV3.2
- new net: R13.2, RV2.3
- new net: C34.1, R18.2
- new net: D12.1 (K), Q5.3 (B), RV1.2
- new net: R12.2, RV1.3
Other:
- moved on the sheet: C21, C22, C23, C24, C25, C26, C27, C28, D10, D11, D8, D9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

Commit message: Driver bias
Parts:
- added C21, C23, C28, C30, C48: 1nF, symbol Device:C_Small
- added C22, C24, C32, C34, C38: 10uF, symbol Device:C_Polarized_Small
- added C25, C26: 30nF, symbol Device:C_Small
- added C36, C41, C42, C50: 100nF, symbol Device:C_Small
- added C44, C46: 84pF, symbol Device:C_Small
- added D11, D13, D9: 1N4148, Diode_THT:D_DO-35_SOD27_P7.62mm_Horizontal, symbol Diode:1N4148
- added D15, D17: 1N4744A, symbol Device:D_Schottky
- added L10, L3, L4: 10uH/1A, symbol Device:L_Small
- added L13, L14: 10uH/100mA, symbol Device:L_Ferrite_Small
- added L5, L6, L7, L8: 10uH, symbol Device:L_Ferrite_Small
- added Q1, Q2, Q8: BD139, Package_TO_SOT_THT:TO-126-3_Vertical, symbol Transistor_BJT:BD139
- added Q11, Q12: IRF630, Package_TO_SOT_THT:TO-220-3_Vertical, symbol Transistor_FET:IRF540N
- added Q5: 2SC5171, Package_TO_SOT_THT:TO-126-3_Vertical, symbol Transistor_BJT:BD139
- added Q6: 2SA1930, Package_TO_SOT_THT:TO-126-3_Vertical, symbol Transistor_BJT:BD140
- added R10, R7, R8, R9: 6k5, symbol Device:R_Small
- added R13, R14: 100R/No ind, symbol Device:R_Small
- added R16: 1R/No ind, symbol Device:R_Small
- added R18: 18k, symbol Device:R_Small
- added R21, R22: 6k8, symbol Device:R_Small
- added R25, R26: 4.7R/No ind, symbol Device:R_Small
- added R29, R30, R36, R38: 100k/No ind, symbol Device:R_Small
- added R33, R34: 125R/No ind, symbol Device:R_Small
- added R39, R40, R41, R42: 33R/No ind, symbol Device:R_Small
- added R5, R6: 345R, symbol Device:R_Small
- added RV1, RV2, RV4: 10k, symbol Device:R_Potentiometer_Trim
- added RV7: 10k - Bias 1, symbol Device:R_Potentiometer_Trim
- added RV8: 10k - Bias 2, symbol Device:R_Potentiometer_Trim
- R19: renamed from R13; value 4k7 -> 6k8
- R20: renamed from R14; value 4k7 -> 6k8
- renumbered C21 to C27, C22 to C29, C23 to C31, C24 to C33, C29 to C35, C30 to C37, C31 to C39, C32 to C40, C34 to C43, C33 to C45, C25 to C47, C27 to C49, C26 to C51, C28 to C52, D9 to D10, D11 to D14, D10 to D16, L6 to L11, L7 to L12, L4 to L15, L5 to L16, L3 to L9, Q4 to Q10, Q1 to Q3, Q2 to Q4, Q5 to Q7, Q3 to Q9, R5 to R11, R6 to R12, R7 to R15, R12 to R17, R8 to R23, R9 to R24, R16 to R27, R17 to R28, R15 to R31, R18 to R32, R11 to R35, R10 to R37, RV1 to RV3, RV2 to RV5, RV3 to RV6
Connections:
- net +24V_Main: now also Q8.2 (C), R18.1
- net GND: now also C21.1, C22.2, C23.1, C24.2, C28.2, C30.1, C30.2, C32.2, C34.1, C34.2, C36.1, C38.2, C41.1, C42.1, C44.2, C46.1, C48.1, C48.2, C50.1, C50.2, D15.2 (A), D17.2 (A), Q11.3 (S), Q12.3 (S), Q6.2 (C), R10.2, R29.1, R30.1, R36.1, R38.1, R8.2, RV4.1, RV7.1, RV8.1
- net at D16.1 (K), R23.2, R27.2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: now also R39.1; no longer Q9.1 (G)
- net at D14.1 (K), R24.2, R28.2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: now also R40.1; no longer Q10.1 (G)
- net at L16.1: now also Q11.2 (D), Q12.2 (D)
- net at R11.1: now also R12.1, L5.2, L7.2
- new net: C25.1, L5.1, Q1.1 (E), R5.2, R8.1
- new net: C25.2, Q1.2 (C), R7.2, RV1.3
- new net: D17.1 (K), R25.2, R29.2, R33.1, R38.2, R41.1
- new net: C46.2, R33.2
- new net: R6.1, RV2.1
- new net: C26.1, L6.1, Q2.1 (E), R10.1, R6.2
- new net: L6.2, L8.2, R13.1, R14.1
- new net: D9.1 (K), Q5.3 (B), R13.2
- new net: D11.1 (K), D9.2 (A), Q5.1 (E), Q6.1 (E), R16.1
- new net: L13.2, L14.2, R16.2, R25.1, R26.1
- new net: C42.2, L14.1, RV8.2
- new net: C28.1, C32.1, L10.2, Q5.2 (C)
- new net: R5.1, RV1.1
- new net: Q1.3 (B), RV1.2
- new net: C26.2, Q2.2 (C), R9.2, RV2.3
- new net: Q2.3 (B), RV2.2
- new net: C44.1, R34.2
- new net: C23.2, C24.1, L4.2, L8.1, R9.1
- new net: D13.1 (K), Q8.3 (B), RV4.2
- new net: R18.2, RV4.3
- new net: D15.1 (K), R26.2, R30.2, R34.1, R36.2, R42.1
- new net: Q12.1 (G), R42.2
- new net: C21.2, C22.1, L3.2, L7.1, R7.1
- new net: R22.2, RV8.3
- new net: Q11.1 (G), R41.2
- new net: Q10.1 (G), R40.2
- new net: C36.2, C38.1, D13.2 (A), Q8.1 (E), R21.1, R22.1
- new net: C41.2, L13.1, RV7.2
- new net: R21.2, RV7.3
- new net: Q9.1 (G), R39.2
- new net: D11.2 (A), Q6.3 (B), R14.2
- new net +15V_Bias_A: L3.1
- new net +15V_Bias_B: L4.1
- new net +15V_DRV_B: L10.1
Other:
- note added: "RF in"
- moved on the sheet: C27, C29, C31, C33, C35, C37, C39, C40, C43, C45, C47, C49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

Commit message: Pre pré drivers work.
Parts:
- added L2: PA In, symbol Intralha.:L_Ferrite_Taped_Coupled_Small
- added Q2, Q3: 2N3866, Package_TO_SOT_THT:TO-39-3, symbol Transistor_BJT:2N2219
- added R48, R49: 3R5/No ind, symbol Device:R_Small
- added R8, R9: 35R/No ind, symbol Device:R_Small
- renumbered C21 to C13, C22 to C14, C23 to C15, C24 to C16, C25 to C17, C26 to C18, C27 to C19, C28 to C20, C29 to C21, C30 to C22, C31 to C23, C32 to C24, C33 to C25, C34 to C26, C35 to C27, C36 to C28, C37 to C29, C38 to C30, C39 to C31, C40 to C32, C41 to C33, C42 to C34, C43 to C35, C44 to C36, C45 to C37, C46 to C38, C47 to C39, C48 to C40, C49 to C41, C50 to C42, C51 to C43, C52 to C44, D9 to D10, D10 to D11, D11 to D12, D12 to D13, D13 to D14, D14 to D15, D15 to D16, D16 to D17, D17 to D18, D8 to D9, Q7 to Q10, Q8 to Q11, Q9 to Q12, Q10 to Q13, Q11 to Q14, Q12 to Q15, Q1 to Q4, Q2 to Q5, Q3 to Q6, Q4 to Q7, Q5 to Q8, Q6 to Q9, R5 to R10, R6 to R11, R7 to R12, R8 to R13, R9 to R14, R10 to R15, R11 to R16, R12 to R17, R13 to R18, R14 to R19, R15 to R20, R16 to R21, R17 to R22, R18 to R23, R19 to R24, R20 to R25, R21 to R26, R22 to R27, R23 to R28, R24 to R29, R25 to R30, R26 to R31, R27 to R32, R28 to R33, R29 to R34, R30 to R35, R31 to R36, R32 to R37, R33 to R38, R34 to R39, R35 to R40, R36 to R41, R37 to R42, R38 to R43, R39 to R44, R40 to R45, R41 to R46, R42 to R47
Connections:
- net +15V_Bias_B is gone; now on net +15V_Main: L4.1
- net +15V_DRV_A is gone; now on net +15V_Main: L9.1
- net +15V_DRV_B is gone; now on net +15V_Main: L10.1
- net +15V_Bias_A renamed +15V_Main
- new net: Q3.1 (E), R48.1
- new net: Q3.2 (B), R9.2
- new net: Q2.1 (E), R49.1
- new net: Q2.2 (B), R8.2

Commit message: Pre pré drivers work II
Parts:
- removed Q3: 2N3866, Package_TO_SOT_THT:TO-39-3, symbol Transistor_BJT:2N2219
- added C47, C49: 100nF, symbol Device:C_Small
- added C48: 74nF, symbol Device:C_Small
- added C50: 10uF, symbol Device:C_Polarized_Small
- added C51: 73nF, symbol Device:C_Small
- added L17: 10uH/1A, symbol Device:L_Small
- L2: value PA In -> DRV In
- R48: value 3R5/No ind -> 1R5/No ind
- R49: value 3R5/No ind -> 10R/No ind
- R8: value 35R/No ind -> 22R/No ind
- R9: value 35R/No ind -> 10k
Connections:
- net +15V_Main: now also L17.1
- net GND: now also R48.1, R9.1, C47.1, C48.1, C49.1, C50.2
- net at R48.2: now also Q2.1 (E), C48.2
- net at L5.2, L7.2, R16.1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: now also R49.1
- net at R9.2: now also Q2.2 (B), R8.2, C47.2
- net at Q2.3 (C): now also C49.2, C50.1, C51.1, L17.2
- net at R8.1: now also L2.4
- net at R49.2: now also C51.2
Other:
- moved on the sheet: L2, Q2

Commit message: PA done.
Parts:
- added C52, C58, C59, C61: 100nF, symbol Device:C_Small
- added C53, C57, C62: 10uF, symbol Device:C_Polarized_Small
- added C54: 285nF, symbol Device:C_Small
- added C55, C56, C60: 74nF, symbol Device:C_Small
- added C63: 73nF, symbol Device:C_Small
- added L18, L19, L20: 10uH/1A, symbol Device:L_Small
- added Q16, Q3: 2N2222A, Package_TO_SOT_THT:TO-18-3, symbol Transistor_BJT:BC107
- added Q17: 2N3866, Package_TO_SOT_THT:TO-39-3, symbol Transistor_BJT:2N2219
- added R50, R56: 5k, symbol Device:R_Small
- added R51, R54: 2k, symbol Device:R_Small
- added R52: 100k, symbol Device:R_Small
- added R53, R57: 735R, symbol Device:R_Small
- added R55: 22R/No ind, symbol Device:R_Small
- added R58: 10k, symbol Device:R_Small
- added R59: 1R5/No ind, symbol Device:R_Small
- added R60: 10R/No ind, symbol Device:R_Small
- added RV10, RV9: 3k5, symbol Device:R_Potentiometer_Trim
Connections:
- net +15V_Main: now also L20.1, R50.2, R56.2
- net GND: now also C52.2, C53.2, C54.2, C57.2, C58.2, C59.1, C60.1, C61.1, C62.2, R52.1, R58.1, R59.1
- net at L6.2, L8.2, R18.1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: now also R60.1
- net at C47.2, Q2.2 (B), R8.2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: now also C52.1, C53.1, L18.2
- net at R8.1: now also C55.2; no longer L2.4
- net at L2.3: now also C56.1
- net at L2.5 (Tap): now also C54.1, R52.2
- new net: Q16.1 (E), R54.1, R57.1
- new net: R54.2, RV10.1
- new net: C56.2, R55.1
- new net: C57.1, C58.1, C59.2, L19.2, Q17.2 (B), R55.2, R58.2
- new net: Q16.3 (C), R56.1, RV10.3
- new net: L19.1, R57.2
- new net: Q16.2 (B), RV10.2
- new net: C60.2, Q17.1 (E), R59.2
- new net: C63.2, R60.2
- new net: Q3.1 (E), R51.1, R53.1
- new net: R51.2, RV9.1
- new net: C61.2, C62.1, C63.1, L20.2, Q17.3 (C)
- new net: C55.1, L2.4
- new net: L18.1, R53.2
- new net: Q3.2 (B), RV9.2
- new net: Q3.3 (C), R50.1, RV9.3
Other:
- moved on the sheet: L2

Commit message: Logical Work
Parts:
- removed L16: PA_Out, symbol Intralha.:L_Ferrite_Taped_Coupled_Small_2
- removed L2: DRV In, symbol Intralha.:L_Ferrite_Taped_Coupled_Small
- added L2: Pre_DRV_In, symbol omega:L_Ferrite_Taped_Coupled_Small
- added L20: PA_Out, symbol omega:L_Ferrite_Taped_Coupled_Small_2
- renumbered C54 to C15, C55 to C16, C56 to C17, C53 to C18, C52 to C19, C57 to C20, C58 to C21, C47 to C22, C59 to C23, C48 to C24, C60 to C25, C49 to C26, C50 to C27, C61 to C28, C62 to C29, C51 to C30, C63 to C31, C13 to C32, C14 to C33, C15 to C34, C16 to C35, C17 to C36, C18 to C37, C19 to C38, C20 to C39, C21 to C40, C22 to C41, C23 to C42, C24 to C43, C25 to C44, C26 to C45, C27 to C46, C28 to C47, C29 to C48, C30 to C49, C31 to C50, C32 to C51, C33 to C52, C34 to C53, C35 to C54, C36 to C55, C37 to C56, C38 to C57, C39 to C58, C40 to C59, C41 to C60, C42 to C61, C43 to C62, C44 to C63, L6 to L10, L7 to L11, L8 to L12, L9 to L13, L10 to L14, L11 to L15, L12 to L16, L13 to L17, L14 to L18, L15 to L19, L18 to L3, L19 to L4, L17 to L5, L20 to L6, L3 to L7, L4 to L8, L5 to L9, Q8 to Q10, Q9 to Q11, Q10 to Q12, Q11 to Q13, Q12 to Q14, Q13 to Q15, Q14 to Q16, Q15 to Q17, Q3 to Q2, Q16 to Q3, Q2 to Q4, Q17 to Q5, Q4 to Q6, Q5 to Q7, Q6 to Q8, Q7 to Q9, R8 to R10, R54 to R11, R55 to R12, R50 to R13, R53 to R14, R56 to R15, R57 to R16, R9 to R17, R58 to R18, R48 to R19, R59 to R20, R49 to R21, R60 to R22, R10 to R23, R11 to R24, R12 to R25, R13 to R26, R14 to R27, R15 to R28, R16 to R29, R17 to R30, R18 to R31, R19 to R32, R20 to R33, R21 to R34, R22 to R35, R23 to R36, R24 to R37, R25 to R38, R26 to R39, R27 to R40, R28 to R41, R29 to R42, R30 to R43, R31 to R44, R32 to R45, R33 to R46, R34 to R47, R35 to R48, R36 to R49, R37 to R50, R38 to R51, R39 to R52, R40 to R53, R41 to R54, R42 to R55, R43 to R56, R44 to R57, R45 to R58, R46 to R59, R47 to R60, R52 to R8, R51 to R9, RV9 to RV1, RV8 to RV10, RV10 to RV2, RV1 to RV3, RV2 to RV4, RV3 to RV5, RV4 to RV6, RV5 to RV7, RV6 to RV8, RV7 to RV9
Connections:
- net GND: now also L20.4
- net at C15.1, R8.2: now also L2.5 (Tap)
- net at Q14.2 (D), Q15.2 (D): now also L20.2
- net at Q16.2 (D), Q17.2 (D): now also L20.1
- net at C16.1: now also L2.4
- net at C62.1, C63.1, L19.2: now also L20.3 (Tap)
- net at C17.1: now also L2.3
- new net LPF_IN: L20.5

Commit message: Logical Work, Mixers II
Parts:
- L2: value Pre_DRV_In -> ~
Connections:
- net +24V_Main: no longer L19.1
- net Pre_DRV_In: now reaches L2.2
- net LPF_IN renamed LPF
- new net +24V_MAIN: L19.1
Changed lines of the file:
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@@
 	(wire
 		(pts
+			(xy 16.51 88.9) (xy 16.51 92.71)
+		)
+		(stroke
+			(width 0)
+			(type default)
+		)
+	)
+	(wire
+		(pts
 			(xy 104.14 113.03) (xy 105.41 113.03)
 		)
@@
 		)
 	)
+	(global_label "LPF"
+		(shape output)
+		(at 273.05 86.36 90)
+		(fields_autoplaced yes)
+		(effects
+			(font
+				(size 0.8 0.8)
+			)
+			(justify left)
+		)
+		(property "Intersheetrefs" "${INTERSHEET_REFS}"
+			(at 273.05 82.3464 90)
+			(effects
+				(font
+					(size 1.27 1.27)
+				)
+				(justify left)
+				(hide yes)
+			)
+		)
+	)
+	(global_label "+24V_MAIN"
+		(shape input)
+		(at 242.57 90.17 90)
+		(fields_autoplaced yes)
+		(effects
+			(font
+				(size 0.8 0.8)
+			)
+			(justify left)
+		)
+		(property "Intersheetrefs" "3"
+			(at 242.57 81.6611 90)
+			(effects
+				(font
+					(size 1.27 1.27)
+				)
+				(justify left)
+				(hide yes)
+			)
+		)
+	)
 	(symbol
 		(lib_id "power:GND")
@@
 	)
 	(symbol
-		(lib_id "power:+12V")
-		(at 273.05 86.36 0)
-		(unit 1)
-		(exclude_from_sim no)
-		(in_bom yes)
-		(on_board yes)
-		(dnp no)
-		(property "Reference" "#PWR0103"
-			(at 273.05 90.17 0)
-			(effects
-				(font
-					(size 1.27 1.27)
-				)
-				(hide yes)
-			)
-		)
-		(property "Value" "LPF_IN"
-			(at 273.812 84.836 0)
-			(effects
-				(font
-					(size 1.27 1.27)
-				)
-				(justify left)
-			)
-		)
-		(property "Footprint" ""
-			(at 273.05 86.36 0)
-			(effects
-				(font
-					(size 1.27 1.27)
-				)
-				(hide yes)
-			)
-		)
-		(property "Datasheet" ""
-			(at 273.05 86.36 0)
-			(effects
-				(font
-					(size 1.27 1.27)
-				)
-				(hide yes)
-			)
-		)
-		(property "Description" "Power symbol creates a global label with name \"+12V\""
-			(at 273.05 86.36 0)
-			(effects
-				(font
-					(size 1.27 1.27)
-				)
-				(hide yes)
-			)
-		)
-		(pin "1"
-		)
-		(instances
-			(project "Omega Radio"
-				(path "/3468ce30-82a7-4087-a7ac-02063723d842/24312ef5-36e6-40ee-ad2e-2d0b81e7182c"
-					(reference "#PWR0103")
-					(unit 1)
-				)
-			)
-		)
-	)
-	(symbol
 		(lib_id "Device:R_Small")
 		(at 232.41 113.03 90)
@@
 	)
 	(symbol
-		(lib_id "power:+12V")
-		(at 242.57 90.17 0)
-		(unit 1)
-		(exclude_from_sim no)
-		(in_bom yes)
-		(on_board yes)
-		(dnp no)
-		(property "Reference" "#PWR094"
-			(at 242.57 93.98 0)
-			(effects
-				(font
-					(size 1.27 1.27)
-				)
-				(hide yes)
-			)
-		)
-		(property "Value" "+24V_Main"
-			(at 235.458 88.646 0)
-			(effects
-				(font
-					(size 1.27 1.27)
-				)
-			)
-		)
-		(property "Footprint" ""
-			(at 242.57 90.17 0)
-			(effects
-				(font
-					(size 1.27 1.27)
-				)
-				(hide yes)
-			)
-		)
-		(property "Datasheet" ""
-			(at 242.57 90.17 0)
-			(effects
-				(font
-					(size 1.27 1.27)
-				)
-				(hide yes)
-			)
-		)
-		(property "Description" "Power symbol creates a global label with name \"+12V\""
-			(at 242.57 90.17 0)
-			(effects
-				(font
-					(size 1.27 1.27)
-				)
-				(hide yes)
-			)
-		)
-		(pin "1"
-		)
-		(instances
-			(project "Omega Radio"
-				(path "/3468ce30-82a7-4087-a7ac-02063723d842/24312ef5-36e6-40ee-ad2e-2d0b81e7182c"
-					(reference "#PWR094")
-					(unit 1)
-				)
-			)
-		)
-	)
-	(symbol
 		(lib_id "Device:R_Small")
 		(at 212.09 140.97 180)
@@
 	)
 	(symbol
+		(lib_id "power:+5VP")
+		(at 16.51 88.9 0)
+		(unit 1)
+		(exclude_from_sim no)
+		(in_bom yes)
+		(on_board yes)
+		(dnp no)
+		(property "Reference" "#PWR0150"
+			(at 16.51 92.71 0)
+			(effects
+				(font
+					(size 1.27 1.27)
+				)
+				(hide yes)
+			)
+		)
+		(property "Value" "Pre_DRV_In"
+			(at 13.97 87.63 90)
+			(effects
+				(font
+					(size 0.8 0.8)
+				)
+			)
+		)
+		(property "Footprint" ""
+			(at 16.51 88.9 0)
+			(effects
+				(font
+					(size 1.27 1.27)
+				)
+				(hide yes)
+			)
+		)
+		(property "Datasheet" ""
+			(at 16.51 88.9 0)
+			(effects
+				(font
+					(size 1.27 1.27)
+				)
+				(hide yes)
+			)
+		)
+		(property "Description" "Power symbol creates a global label with name \"+5VP\""
+			(at 16.51 88.9 0)
+			(effects
+				(font
+					(size 1.27 1.27)
+				)
+				(hide yes)
+			)
+		)
+		(pin "1"
+		)
+		(instances
+			(project ""
+				(path "/3468ce30-82a7-4087-a7ac-02063723d842/24312ef5-36e6-40ee-ad2e-2d0b81e7182c"
+					(reference "#PWR0150")
+					(unit 1)
+				)
+			)
+		)
+	)
+	(symbol
 		(lib_id "power:GND")
 		(at 273.05 99.06 0)
@@
 		(dnp no)
 		(property "Reference" "L2"
-			(at 17.78 90.678 90)
+			(at 14.732 95.504 90)
 			(effects
 				(font
@@
 			)
 		)
-		(property "Value" "Pre_DRV_In"
-			(at 13.462 100.33 0)
+		(property "Value" "~"
+			(at 15.494 102.616 0)
 			(effects
 				(font
@@
 				)
 				(justify left)
+				(hide yes)
 			)
 		)
