File: Power.kicad_sch (KiCad schematic)
At the start: 38 parts, among them SW2 POWER SWITCH, U1 LM7805_TO220

Commit message: Driver done.
Parts:
- renumbered C1 to C10, C2 to C11, C3 to C12, C6 to C13, C4 to C14, C7 to C15, C8 to C16, C9 to C17, C10 to C2, C11 to C3, C12 to C4, C13 to C5, C14 to C6, C15 to C7, C16 to C8, C17 to C9, D3 to D1, D4 to D2, D5 to D3, D6 to D4, D7 to D5, D1 to D6, D2 to D7, FL2 to FL1, FL1 to FL2, TP4 to TP1, TP1 to TP2, TP2 to TP3, TP3 to TP4, U1 to U2

Commit message: huge modification of the project.
Parts:
- removed C10: 330nF, symbol Device:C
- removed C11: 450uF, symbol Device:C_Polarized
- removed C12: 100nF, symbol Device:C
- removed C13, C17: 100nF, symbol Device:C_Small
- removed C14: 100uF/25V, symbol Device:C_Polarized
- removed C15, C16: 100uF, symbol Device:C_Polarized_Small
- removed C2: CY- 4,7nF, symbol Device:C_Small
- removed CHASSIS1: TestPoint_Alt, symbol Connector:TestPoint_Alt
- removed D6: 1N5819, Diode_THT:D_DO-41_SOD81_P10.16mm_Horizontal, symbol Diode:1N5819
- removed D7: P6KE6.8A, Diode_THT:D_P600_R-6_P20.00mm_Horizontal, symbol Diode:5KPxxA
- removed FB1: ≈ 600 Ω @ 100 MHz, symbol Device:FerriteBead_Small
- removed FL2: ≥600 Ω @100 MHz,, Inductor_THT:L_CommonMode_PulseElectronics_PH9455x105NL_1, symbol Filter:Choke_CommonMode_PulseElectronics_PH9455x105NL
- removed TP2: GND_LM7895, symbol Connector:TestPoint
- removed TP3: 5V_DIG, symbol Connector:TestPoint
- removed TP4: 5V_DIG2, symbol Connector:TestPoint
- removed U2: LM7805_TO220, Package_TO_SOT_THT:TO-220-3_Vertical, symbol Regulator_Linear:LM7805_TO220
- added C10: CY- 4,7nF, symbol Device:C_Small
- added C11, C12, C15: 100nF, symbol Device:C_Small
- added C13, C2: 1000uF, symbol Device:C_Polarized_Small
- added C14: 470uF, symbol Device:C_Polarized_Small
- added CHASSIS: TestPoint_Alt, symbol Connector:TestPoint_Alt
- added D6: 1N4002, Diode_THT:D_DO-41_SOD81_P10.16mm_Horizontal, symbol Diode:1N4002
- added L11: 100uH/1A, symbol Device:L_Small
- added U2: LM7815C, Package_TO_SOT_THT:TO-220-3_Vertical, symbol Regulator_Linear:LM7815_TO220
- D2: value BZT52C15 -> BZT52C27
- D3: value P6KE18A -> P6KE33A
- D4: value MBR3045 -> MBR3060
- R1: value 1k -> 1k-1/4W
- R2: value 150R -> 150R/0.5W
- R3: value 10R -> 10R - 1/2W
- R4: value 1k5 -> 100R/1W
- TP1: value +12V_SW -> +24_SW
- renumbered CHASSIS2 to CHASSIS
Connections:
- net +12V_IN is gone; now on an unnamed net: SW2.2 (B)
- net GND: now also C9.1, C11.2, C12.2, C13.2, C14.2, C15.2, C2.2, U2.2 (GND)
- net at C3.1, C4.1, C5.1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: no longer SW2.1 (A)
- net +12V_SW renamed +24V_Main
- net +24V_Main: now also C10.2, L11.1
- net GND_IN renamed GNDP.
- net GNDP.: no longer C9.1, D2.2 (A), R1.2
- new net: D2.2 (A), R1.2
- new net: C10.1, CHASSIS.1
- new net: C14.1, C15.1, D6.1 (K), L11.2, U2.1 (VI)
- new net +15V_DRV_A: C11.1, C12.1, C13.1, C2.1, D6.2 (A), U2.3 (VO)
- new net +24V_IN: SW2.1 (A)
Other:
- note added: "All caps >= 50V"
- moved on the sheet: C3, C4, C5, C6, C7, C8, C9, CHASSIS, D1, D2, D3, D4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

Commit message: PA reformulation
Parts:
- removed C9: CY+ 4,7nF, symbol Device:C_Small
- renumbered C5 to C10, C4 to C11, C7 to C12, C6 to C13, C10 to C14, C15 to C2, C14 to C3, C12 to C4, C11 to C5, C13 to C6, C2 to C7, C3 to C9, CHASSIS to CHASSIS1, CHASSIS to CHASSIS2, D6 to D1, D4 to D2, D2 to D3, D5 to D4, D1 to D5, D3 to D6, L11 to L1, R4 to R3, R3 to R4
Connections:
- net GND: now also CHASSIS2.1
- net +24V_IN renamed +24V_P
Other:
- moved on the sheet: C13, C14, CHASSIS1, CHASSIS2, D6

Commit message: Bias Work
Parts:
- added C12: 1000uF, symbol Device:C_Polarized_Small
- added C13: 10uF, symbol Device:C_Polarized_Small
- added C3, C8, C9: 100nF, symbol Device:C_Small
- added C5: 470uF, symbol Device:C_Polarized_Small
- added D2: 1N4002, Diode_THT:D_DO-41_SOD81_P10.16mm_Horizontal, symbol Diode:1N4002
- added L2: 100uH/1A, symbol Device:L_Small
- added U3: LM7815C, Package_TO_SOT_THT:TO-220-3_Vertical, symbol Regulator_Linear:LM7815_TO220
- C11: renamed from C7; value 1000uF -> 10uF
- renumbered C6 to C10, C8 to C14, C9 to C15, C10 to C16, C11 to C17, C12 to C18, C13 to C19, C14 to C20, C3 to C4, C4 to C6, C5 to C7, D2 to D3, D3 to D4, D4 to D5, D5 to D6, D6 to D7
Connections:
- net +24V_Main: now also L2.1
- net GND: now also C12.2, C13.2, C3.2, C5.2, C8.2, C9.2, U3.2 (GND)
- net +15V_DRV_A renamed +15V_Bias_A
- new net: C3.1, C5.1, D2.1 (K), L2.2, U3.1 (VI)
- new net +15V_Bias_B: C12.1, C13.1, C8.1, C9.1, D2.2 (A), U3.3 (VO)

Commit message: Pre pré drivers work.
Parts:
- removed C11, C13: 10uF, symbol Device:C_Polarized_Small
- removed C12: 1000uF, symbol Device:C_Polarized_Small
- removed C3, C7, C8, C9: 100nF, symbol Device:C_Small
- removed C5: 470uF, symbol Device:C_Polarized_Small
- removed D2: 1N4002, Diode_THT:D_DO-41_SOD81_P10.16mm_Horizontal, symbol Diode:1N4002
- removed L2: 100uH/1A, symbol Device:L_Small
- removed U3: LM7815C, Package_TO_SOT_THT:TO-220-3_Vertical, symbol Regulator_Linear:LM7815_TO220
- added C45: 10uF, symbol Device:C_Polarized_Small
- added C46: 100nF, symbol Device:C_Small
- added D2: 1N5404, Diode_THT:D_DO-201AD_P15.24mm_Horizontal, symbol Diode:1N5404
- added D4: 1N4148, Diode_THT:D_DO-35_SOD27_P7.62mm_Horizontal, symbol Diode:1N4148
- added Q1: TIP35C, Package_TO_SOT_THT:TO-247-3_Vertical, symbol Transistor_BJT:TIP3055G
- added R2: 0.20R/5W, symbol Device:R_Small
- added R3: 1k/0.25W, symbol Device:R_Small
- added R4: 56R/2W, symbol Device:R_Small
- L1: value 100uH/1A -> 100uH/5A
- renumbered C18 to C10, C19 to C11, C20 to C12, C4 to C3, C6 to C4, C14 to C5, C10 to C6, C15 to C7, C16 to C8, C17 to C9, D4 to D5, D5 to D6, D6 to D7, D7 to D8, R2 to R5, R3 to R6, R4 to R7
Connections:
- net GND: now also C45.2, C46.2, D4.2 (A); no longer U2.2 (GND)
- net at C2.1, C3.1, D1.1 (K)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: now also D2.1 (K), Q1.2 (C)
- net +15V_Bias_A: no longer names the net of D1.2 (A), U2.3 (VO)
- net +15V_Bias_A: now also C45.1, C46.1, R4.1; no longer C4.1, C6.1
- new net: Q1.1 (B), R3.1, R4.2
- new net: D2.2 (A), Q1.3 (E), R2.1
- new net: D4.1 (K), U2.2 (GND)
- new net +15V_Main: C4.1, C6.1, R2.2, R3.2
Other:
- moved on the sheet: C2, C3, C4, C6, D1, L1, U2

Commit message: Logical Work
Parts:
- renumbered C8 to C10, C9 to C11, C10 to C12, C11 to C13, C12 to C14, C45 to C4, C46 to C6, C4 to C7, C7 to C8, C6 to C9, D3 to D1, D5 to D2, D2 to D3, D1 to D4, D4 to D5, R5 to R2, R2 to R3, R6 to R4, R4 to R5, R3 to R6

Commit message: Logical Work, Mixers II
Parts:
- removed TP1: +24_SW, symbol Connector:TestPoint
Connections:
- net GNDP. is gone; now on net GND_S: C10.2, C11.2, C5.2, D1.2 (A), D6.2 (A), D7.1 (K), FL1.2, R4.2, R7.2
- net +24V_Main: no longer C12.1, C13.1, C14.2, D8.1 (A1), FL1.4
- net +24V_P renamed GND_S
- new net +24V_MAIN: C12.1, C13.1, C14.2, D8.1 (A1), FL1.4
