File: rf_if.kicad_sch (KiCad schematic)
At the start: 1 part

Commit message: Logical Work
Parts:
- removed U3: ~, symbol Intralha.:Adafruit_Si5351
- added C76, C78: 100nF, symbol Device:C_Small
- added C77, C79: 10uF, symbol Device:C_Polarized_Small
- added R61: 33R, symbol Device:R_Small
- added R62, R63: 10k, symbol Device:R_Small
- added U3: Adafruit_Si5351, symbol omega:Adafruit_Si5351
- added U4: 74LVC74, symbol omega:74LVC74
- added U5: 74HCT244, symbol 74xx:74HCT244
- added U6, U7: 74HC4066, symbol omega:74HC4066
Connections:
- new net: R63.2, U4.13 (2CLR)
- new net: R62.2, U4.1 (CLR)
- new net: R61.1, U4.11 (2CK), U4.3 (1CK)
- new net: R61.2, U3. (GND2)
- new net: U4.12 (2D), U4.5 (1Q)
- new net: U4.2 (1D), U4.9 (2Q)
- new net +3.3V: C76.1, C77.1, R62.1, R63.1, U4.10 (2PR), U4.14 (VCC), U4.4 (1PR)
- new net +5V: C78.1, C79.1, U5.20 (VCC)
- new net GND: C76.2, C77.2, C78.2, C79.2, U4.7 (GND), U5.1 (1OE), U5.10 (GND), U5.19 (2OE)
- no-connect marks 0 -> 2

Commit message: Logical Work, Mixers
Connections:
- net +3.3V: now also R62.2; no longer R62.1
- net at R63.2: now also U4.1 (CLR); no longer U4.13 (2CLR)
- net CLK0: now reaches R61.1, U4.11 (2CK), U4.3 (1CK)
- net LO_1: now reaches U4.12 (2D), U4.5 (1Q)
- net LO_1: now also U5.16 (1Y1), U5.4 (1A1)
- net LO_2: now reaches U4.2 (1D), U4.9 (2Q)
- net LO_2: now also U5.15 (2A1), U5.5 (2Y1)
- net LO_1_INV: now reaches U4.6 (1#Q)
- net LO_1_INV: now also U5.14 (1Y2), U5.6 (1A2)
- net LO_2_INV: now reaches U4.8 (2#Q)
- net LO_2_INV: now also U5.13 (2A2), U5.7 (2Y2)
- new net: R62.1, U4.13 (2CLR)
- no-connect marks 2 -> 0
Other:
- moved on the sheet: C76, C77, C78, C79, R61, R62, R63, U3, U4, U5

Commit message: Logical Work, Mixers II
Parts:
- added C80, C82, C84: 100nF, symbol Device:C_Small
- added C81, C83, C85: 10uF, symbol Device:C_Polarized_Small
- added R64, R65: 100R, symbol Device:R_Small
- added R66, R67: 10k, symbol Device:R_Small
- added U8: LM358, symbol omega:LM358
Connections:
- net +5V: now also U6.14 (VCC), U7.14 (VCC), C80.1, C81.1, C82.1, C83.1, C84.1, C85.1, U8.8 (V+)
- net GND: now also U6.7 (GND), U7.7 (GND), C80.2, C81.2, C82.2, C83.2, C84.2, C85.2, U8.3 (IN1+), U8.4 (V-)
- net LO_1: now also R64.2
- net LO_1_INV: now also R65.1
- net +I_Signal: now reaches U6.1 (1Y)
- net +I_Signal: now also R66.1
- net at U6.13 (1E): now also R64.1
- net RF_Channel_1: now reaches U6.2 (1Z)
- net RF_Channel_1: now also U6.3 (2Z)
- net -I_Signal: now reaches U6.4 (2Y)
- net at U6.5 (2E): now also R65.2
- new net: R66.2, R67.1, U8.2 (IN1-)
- new net: R67.2, U8.1 (OUT1)
- new net: U8.11 (NC), U8.4 (V-)
Other:
- note added: "CHANELL_1"
- moved on the sheet: C76, C77, C78, C79, R61, R62, R63, U3, U4, U5, U6, U7

Commit message: Logical Work, Mixers III
Parts:
- added C86: 220nF, symbol Device:C_Small
- added R68, R69: 10k-1/4W, symbol Device:R_Small
- added R70: 100k-1/4W, symbol Device:R_Small
- added R71, R72: 100R, symbol Device:R_Small
Connections:
- net -I_Signal is gone; now on net RF_CHANELL_1: U6.4 (2Y)
- net +5V: now also R68.1
- net GND: now also R69.1; no longer U8.3 (IN1+)
- net LO_1: now also R71.2
- net LO_1_INV: now also R72.1
- net VREF: now reaches U8.5 (IN2+)
- net VREF: now also U8.3 (IN1+), R68.2, R69.2, R70.1
- net -I _SIGNAL: now reaches U6.10 (4Z)
- net -I _SIGNAL: now also U6.3 (2Z)
- net RF_CHANELL_1: now reaches U6.11 (4Y)
- net RF_CHANELL_1: now also U6.1 (1Y), U6.8 (3Y)
- net at U6.12 (4E): now also R71.1
- net at U6.6 (3E): now also R72.2
- net +I _SIGNAL: now reaches U6.9 (3Z)
- net +I _SIGNAL: now also U6.2 (1Z)
- net +I_Signal renamed I_REF
- net I_REF: now also C86.1, R70.2; no longer U6.1 (1Y)
- removed net RF_Channel_1: U6.2 (1Z), U6.3 (2Z)
- new net +I_SOUND: C86.2
Other:
- note added: "I MIXER"
- note removed: "CHANELL_1"
- moved on the sheet: C76, C77, C78, C79, C80, C81, C82, C83, C84, C85, R61, R62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

Commit message: Logical Work, Mixers IV
Parts:
- added C89: 220nF, symbol Device:C_Small
- added R73, R74, R75, R76: 100R, symbol Device:R_Small
- added R79: 100k-1/4W, symbol Device:R_Small
- added R80, R81: 10k, symbol Device:R_Small
Connections:
- net I_REF is gone; now on net I _REF: C86.1, R66.1, R70.2
- net -I _SIGNAL: now also R67.2, U8.1 (OUT1)
- net LO_2: now also R75.2, R76.2
- net LO_2_INV: now also R73.1, R74.1
- net VREF: now also R79.1
- net RF_CHANELL_2: now reaches U7.1 (1Y)
- net RF_CHANELL_2: now also U7.11 (4Y), U7.4 (2Y), U7.8 (3Y)
- net -Q _SIGNAL: now reaches U7.10 (4Z)
- net -Q _SIGNAL: now also U7.3 (2Z), U8.7 (OUT2), R80.1
- net at U7.12 (4E): now also R76.1
- net at U7.13 (1E): now also R75.1
- net Q _REF: now reaches U7.2 (1Z)
- net Q _REF: now also U7.9 (3Z), C89.1, R79.2, R81.2
- net at U7.5 (2E): now also R73.2
- net at U7.6 (3E): now also R74.2
- net at U8.6 (IN2-): now also R80.2, R81.1
- net +I _SIGNAL renamed I _REF
- net +I_SOUND renamed +I _SOUND
- new net +Q_SOUND: C89.2
Other:
- note added: "II MIXER"
- moved on the sheet: C76, C77, C78, C79, C80, C81, R61, R62, R63, R64, R65, R66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
