File: BPF.kicad_sch (KiCad schematic)
At the start: 16 parts

Commit message: BPF Work 2
Parts:
- added C45: 410pF, symbol Device:C_Small
- added C46: 1nF, symbol Device:C_Small
- added C48: 79pF, symbol Device:C_Small
- added C49: 298pF, symbol Device:C_Small
- added C52: 409pF, symbol Device:C_Small
- added C53: 290pF, symbol Device:C_Small
- added C55: 248pF, symbol Device:C_Small
- added C56: 51pF, symbol Device:C_Small
- added L10: 745nH, symbol Device:L_Small
- added L12, L19: 1uH, symbol Device:L_Small
- added L13: 2.5uH, symbol Device:L_Small
- added L16: 607nH, symbol Device:L_Small
- added L17: 128nH, symbol Device:L_Small
- added L20: 726nH, symbol Device:L_Small
- added L9: 198nH, symbol Device:L_Small
- added Q17, Q18, Q19, Q20, Q21, Q22, Q23, Q24, Q25, Q26, Q27, Q28, Q29, Q30, Q31, Q32: BC548, Package_TO_SOT_THT:TO-92_Inline, symbol Transistor_BJT:BC548
- renumbered C106 to C37, C100 to C38, C104 to C39, C102 to C40, C107 to C41, C101 to C42, C105 to C43, C103 to C44, L36 to L1, L30 to L2, L34 to L3, L32 to L4, L37 to L5, L31 to L6, L35 to L7, L33 to L8
Connections:
- net GND: now also C45.1, C46.1, C52.1, C53.1, L10.2, L16.2, L17.2, L9.2
- net at C38.2, C42.2, L2.1: now also Q19.3 (E)
- net at L8.2: now also Q27.3 (E)
- net at C39.2, C43.2, L3.1: now also Q21.3 (E)
- net at C40.2, C44.2, L4.1: now also Q20.3 (E)
- net at L7.2: now also Q28.3 (E)
- net at L6.2: now also Q26.3 (E)
- net at C37.2, C41.2, L1.1: now also Q17.3 (E)
- net at L5.2: now also Q18.3 (E)
- new net: Q29.1 (C), Q29.2 (B)
- new net: C46.2, C49.2, L10.1, Q29.3 (E)
- new net: C52.2, C55.2, L16.1, Q30.3 (E)
- new net: Q17.1 (C), Q17.2 (B)
- new net: Q26.1 (C), Q26.2 (B)
- new net: Q23.1 (C), Q23.2 (B)
- new net: L19.2, Q23.3 (E)
- new net: Q28.1 (C), Q28.2 (B)
- new net: C45.2, C48.2, L9.1, Q31.3 (E)
- new net: C53.2, C56.2, L17.1, Q32.3 (E)
- new net: Q25.1 (C), Q25.2 (B)
- new net: L20.2, Q25.3 (E)
- new net: Q21.1 (C), Q21.2 (B)
- new net: Q27.1 (C), Q27.2 (B)
- new net: C48.1, L12.1
- new net: L12.2, Q24.3 (E)
- new net: Q19.1 (C), Q19.2 (B)
- new net: Q31.1 (C), Q31.2 (B)
- new net: C56.1, L20.1
- new net: C55.1, L19.1
- new net: Q24.1 (C), Q24.2 (B)
- new net: Q32.1 (C), Q32.2 (B)
- new net: Q20.1 (C), Q20.2 (B)
- new net: Q18.1 (C), Q18.2 (B)
- new net: Q22.1 (C), Q22.2 (B)
- new net: L13.2, Q22.3 (E)
- new net: C49.1, L13.1
- new net: Q30.1 (C), Q30.2 (B)
Other:
- note added: "BPF1 - 130kHz - 400kHz"
- note added: "BPF2 - 400kHz - 1.8MHz"
- note added: "BPF3 - 1.8MHz - 2.5MHz"
- note added: "BPF4 - 2.5MHz - 4.7MHz"
- note added: "BPF5 - 4.7MHz - 7.5MHz"
- note added: "BPF6 - 7.5MHz - 14.5MHz"
- note added: "BPF7 - 14.5MHz - 21.5MHz"
- note added: "BPF8 - 21.5MHz - 33MHz"
- note removed: "1.8MHz - 2.5MHz"
- note removed: "130kHz - 400kHz"
- note removed: "2.5MHz - 4.7MHz"
- note removed: "400kHz - 1.8MHz"
- moved on the sheet: C37, C38, C39, C40, C41, C42, C43, C44, L1, L2, L3, L4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

Commit message: BPF Work 3
Parts:
- removed Q23, Q24, Q25: BC548, Package_TO_SOT_THT:TO-92_Inline, symbol Transistor_BJT:BC548
- added C37, C38, C39, C40, C57, C58, C59, C60, C61, C62, C63, C76, C77, C78, C79, C84: 220nF, symbol Device:C_Small
- added C41, C42, C43, C48, C64, C65, C67, C80: 10uF, symbol Device:C_Polarized_Small
- added C46, C47, C49, C52, C68, C70, C72, C82: 10nF, symbol Device:C_Small
- added L13: 8.2uH, symbol Device:L_Small
- added L16: 5.6uH, symbol Device:L_Small
- added L18: 2.7uH, symbol Device:L_Small
- added L23: 1.8uH, symbol Device:L_Small
- added L3: 470uH, symbol Device:L_Small
- added L4: 100uH, symbol Device:L_Small
- added L5: 22uH, symbol Device:L_Small
- added L7: 18uH, symbol Device:L_Small
- added Q13, Q14, Q16: BC548, Package_TO_SOT_THT:TO-92_Inline, symbol Transistor_BJT:BC548
- added R26, R27, R28, R29, R30, R31, R32, R33: 1k2-1/4W, symbol Device:R_Small
- renumbered C37 to C44, C38 to C45, C40 to C50, C39 to C51, C41 to C53, C42 to C54, C44 to C55, C43 to C56, C46 to C66, C45 to C69, C52 to C71, C49 to C73, C48 to C74, C55 to C75, C53 to C81, C56 to C83, L6 to L10, L8 to L11, L7 to L12, L10 to L14, L9 to L15, L16 to L17, L13 to L19, L12 to L20, L19 to L21, L17 to L22, L20 to L24, L4 to L6, L3 to L8, L5 to L9, Q17 to Q1, Q30 to Q10, Q31 to Q11, Q22 to Q12, Q32 to Q15, Q19 to Q2, Q20 to Q3, Q21 to Q4, Q26 to Q5, Q18 to Q6, Q27 to Q7, Q28 to Q8, Q29 to Q9
Connections:
- net GND: now also C41.2, C42.2, C43.2, C46.2, C47.2, C48.2, C49.2, C52.2, C64.2, C65.2, C67.2, C68.2, C70.2, C72.2, C80.2, C82.2
- net at Q9.1 (C), Q9.2 (B): now also Q12.1 (C), Q12.2 (B), C61.1, C76.2, L13.2
- net at Q1.1 (C), Q1.2 (B): now also Q6.1 (C), Q6.2 (B), C37.1, C57.2, L3.2
- net at Q5.1 (C), Q5.2 (B): now also Q2.1 (C), Q2.2 (B), C38.1, C58.2, L4.2
- net at L21.2: now also Q14.3 (E)
- net at Q8.1 (C), Q8.2 (B): now also Q4.1 (C), Q4.2 (B), C40.1, C60.2, L7.2
- net at L24.2: now also Q16.3 (E)
- net at Q7.1 (C), Q7.2 (B): now also Q3.1 (C), Q3.2 (B), C39.1, C59.2, L5.2
- net at L20.2: now also Q13.3 (E)
- net at Q11.1 (C), Q11.2 (B): now also C63.1, C77.2, L18.2, Q13.1 (C), Q13.2 (B)
- net at Q15.1 (C), Q15.2 (B): now also C79.1, C84.2, L23.2, Q16.1 (C), Q16.2 (B)
- net at Q10.1 (C), Q10.2 (B): now also C62.1, C78.2, L16.2, Q14.1 (C), Q14.2 (B)
- new net: C65.1, C70.1, L16.1, R31.2
- new net: C64.1, C68.1, L13.1, R30.2
- new net: C41.1, C46.1, L3.1, R26.2
- new net: C67.1, C72.1, L18.1, R32.2
- new net: C43.1, C49.1, L5.1, R28.2
- new net: C42.1, C47.1, L4.1, R27.2
- new net: C48.1, C52.1, L7.1, R29.2
- new net: C80.1, C82.1, L23.1, R33.2
- new net BPF1_12V: R26.1
- new net BPF2_12V: R27.1
- new net BPF3_12V: R28.1
- new net BPF4_12V: R29.1
- new net BPF5_12V: R30.1
- new net BPF6_12V: R31.1
- new net BPF7_12V: R32.1
- new net BPF8_12V: R33.1
- new net BPF_IN: C37.2, C38.2, C39.2, C40.2, C61.2, C62.2, C63.2, C79.2
- new net BPF_OUT: C57.1, C58.1, C59.1, C60.1, C76.1, C77.1, C78.1, C84.1
Other:
- moved on the sheet: C44, C45, C50, C51, C53, C54, C55, C56, C66, C69, C71, C73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

Commit message: Rf RX amplifier, BPF RX
Parts:
- renumbered C37 to C48, C38 to C49, C39 to C50, C40 to C51, C41 to C52, C42 to C53, C43 to C54, C44 to C55, C45 to C56, C46 to C57, C47 to C58, C48 to C59, C49 to C60, C50 to C61, C51 to C62, C52 to C63, C53 to C64, C54 to C65, C55 to C66, C56 to C67, C57 to C68, C58 to C69, C59 to C70, C60 to C71, C61 to C72, C62 to C73, C63 to C74, C64 to C75, C65 to C76, C66 to C77, C67 to C78, C68 to C79, C69 to C80, C70 to C81, C71 to C82, C72 to C83, C73 to C84, C74 to C85, C75 to C86, C76 to C87, C77 to C88, C78 to C89, C79 to C90, C80 to C91, C81 to C92, C82 to C93, C83 to C94, C84 to C95, L7 to L10, L8 to L11, L9 to L12, L10 to L13, L11 to L14, L12 to L15, L13 to L16, L14 to L17, L15 to L18, L16 to L19, L17 to L20, L18 to L21, L19 to L22, L20 to L23, L21 to L24, L22 to L25, L23 to L26, L24 to L27, L1 to L4, L2 to L5, L3 to L6, L4 to L7, L5 to L8, L6 to L9, Q8 to Q10, Q9 to Q11, Q10 to Q12, Q11 to Q13, Q12 to Q14, Q13 to Q15, Q14 to Q16, Q15 to Q17, Q16 to Q18, Q1 to Q3, Q2 to Q4, Q3 to Q5, Q4 to Q6, Q5 to Q7, Q6 to Q8, Q7 to Q9, R26 to R37, R27 to R38, R28 to R39, R29 to R40, R30 to R41, R31 to R42, R32 to R43, R33 to R44

Commit message: RF Gain
Parts:
- renumbered C95 to C100, C48 to C53, C49 to C54, C50 to C55, C51 to C56, C52 to C57, C53 to C58, C54 to C59, C55 to C60, C56 to C61, C57 to C62, C58 to C63, C59 to C64, C60 to C65, C61 to C66, C62 to C67, C63 to C68, C64 to C69, C65 to C70, C66 to C71, C67 to C72, C68 to C73, C69 to C74, C70 to C75, C71 to C76, C72 to C77, C73 to C78, C74 to C79, C75 to C80, C76 to C81, C77 to C82, C78 to C83, C79 to C84, C80 to C85, C81 to C86, C82 to C87, C83 to C88, C84 to C89, C85 to C90, C86 to C91, C87 to C92, C88 to C93, C89 to C94, C90 to C95, C91 to C96, C92 to C97, C93 to C98, C94 to C99, Q9 to Q10, Q10 to Q11, Q11 to Q12, Q12 to Q13, Q13 to Q14, Q14 to Q15, Q15 to Q16, Q16 to Q17, Q17 to Q18, Q18 to Q19, Q3 to Q4, Q4 to Q5, Q5 to Q6, Q6 to Q7, Q7 to Q8, Q8 to Q9, R37 to R44, R38 to R45, R39 to R46, R40 to R47, R41 to R48, R42 to R49, R43 to R50, R44 to R51

Commit message: AGC Work
Parts:
- renumbered Q9 to Q10, Q10 to Q11, Q11 to Q12, Q12 to Q13, Q13 to Q14, Q14 to Q15, Q15 to Q16, Q16 to Q17, Q17 to Q18, Q18 to Q19, Q19 to Q20, Q4 to Q5, Q5 to Q6, Q6 to Q7, Q7 to Q8, Q8 to Q9
Changed lines of the file:
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@@
 		(dnp no)
 		(fields_autoplaced yes)
-		(property "Reference" "Q12"
+		(property "Reference" "Q13"
 			(at 135.89 48.2599 0)
 			(effects
@@
 			(project "Omega Radio"
 				(path "/3468ce30-82a7-4087-a7ac-02063723d842/ec53c5ee-9461-45e2-ad09-a1b0259ff68e"
-					(reference "Q12")
+					(reference "Q13")
 					(unit 1)
 				)
@@
 		(dnp no)
 		(fields_autoplaced yes)
-		(property "Reference" "Q4"
+		(property "Reference" "Q5"
 			(at 41.91 31.7499 0)
 			(effects
@@
 			(project ""
 				(path "/3468ce30-82a7-4087-a7ac-02063723d842/ec53c5ee-9461-45e2-ad09-a1b0259ff68e"
-					(reference "Q4")
+					(reference "Q5")
 					(unit 1)
 				)
@@
 		(on_board yes)
 		(dnp no)
-		(property "Reference" "Q8"
+		(property "Reference" "Q9"
 			(at 92.964 74.676 0)
 			(effects
@@
 			(project "Omega Radio"
 				(path "/3468ce30-82a7-4087-a7ac-02063723d842/ec53c5ee-9461-45e2-ad09-a1b0259ff68e"
-					(reference "Q8")
+					(reference "Q9")
 					(unit 1)
 				)
@@
 		(on_board yes)
 		(dnp no)
-		(property "Reference" "Q11"
+		(property "Reference" "Q12"
 			(at 99.314 163.322 0)
 			(effects
@@
 			(project "Omega Radio"
 				(path "/3468ce30-82a7-4087-a7ac-02063723d842/ec53c5ee-9461-45e2-ad09-a1b0259ff68e"
-					(reference "Q11")
+					(reference "Q12")
 					(unit 1)
 				)
@@
 		(on_board yes)
 		(dnp no)
-		(property "Reference" "Q17"
+		(property "Reference" "Q18"
 			(at 188.976 97.028 0)
 			(effects
@@
 			(project "Omega Radio"
 				(path "/3468ce30-82a7-4087-a7ac-02063723d842/ec53c5ee-9461-45e2-ad09-a1b0259ff68e"
-					(reference "Q17")
+					(reference "Q18")
 					(unit 1)
 				)
@@
 		(dnp no)
 		(fields_autoplaced yes)
-		(property "Reference" "Q7"
+		(property "Reference" "Q8"
 			(at 52.07 160.0199 0)
 			(effects
@@
 			(project "Omega Radio"
 				(path "/3468ce30-82a7-4087-a7ac-02063723d842/ec53c5ee-9461-45e2-ad09-a1b0259ff68e"
-					(reference "Q7")
+					(reference "Q8")
 					(unit 1)
 				)
@@
 		(on_board yes)
 		(dnp no)
-		(property "Reference" "Q10"
+		(property "Reference" "Q11"
 			(at 94.996 119.38 0)
 			(effects
@@
 			(project "Omega Radio"
 				(path "/3468ce30-82a7-4087-a7ac-02063723d842/ec53c5ee-9461-45e2-ad09-a1b0259ff68e"
-					(reference "Q10")
+					(reference "Q11")
 					(unit 1)
 				)
@@
 		(dnp no)
 		(fields_autoplaced yes)
-		(property "Reference" "Q5"
+		(property "Reference" "Q6"
 			(at 41.91 69.8499 0)
 			(effects
@@
 			(project "Omega Radio"
 				(path "/3468ce30-82a7-4087-a7ac-02063723d842/ec53c5ee-9461-45e2-ad09-a1b0259ff68e"
-					(reference "Q5")
+					(reference "Q6")
 					(unit 1)
 				)
@@
 		(dnp no)
 		(fields_autoplaced yes)
-		(property "Reference" "Q14"
+		(property "Reference" "Q15"
 			(at 139.7 139.6999 0)
 			(effects
@@
 			(project "Omega Radio"
 				(path "/3468ce30-82a7-4087-a7ac-02063723d842/ec53c5ee-9461-45e2-ad09-a1b0259ff68e"
-					(reference "Q14")
+					(reference "Q15")
 					(unit 1)
 				)
@@
 		(on_board yes)
 		(dnp no)
-		(property "Reference" "Q19"
+		(property "Reference" "Q20"
 			(at 266.446 50.038 0)
 			(effects
@@
 			(project "Omega Radio"
 				(path "/3468ce30-82a7-4087-a7ac-02063723d842/ec53c5ee-9461-45e2-ad09-a1b0259ff68e"
-					(reference "Q19")
+					(reference "Q20")
 					(unit 1)
 				)
@@
 		(on_board yes)
 		(dnp no)
-		(property "Reference" "Q16"
+		(property "Reference" "Q17"
 			(at 185.166 144.018 0)
 			(effects
@@
 			(project "Omega Radio"
 				(path "/3468ce30-82a7-4087-a7ac-02063723d842/ec53c5ee-9461-45e2-ad09-a1b0259ff68e"
-					(reference "Q16")
+					(reference "Q17")
 					(unit 1)
 				)
@@
 		(dnp no)
 		(fields_autoplaced yes)
-		(property "Reference" "Q18"
+		(property "Reference" "Q19"
 			(at 222.25 45.7199 0)
 			(effects
@@
 			(project "Omega Radio"
 				(path "/3468ce30-82a7-4087-a7ac-02063723d842/ec53c5ee-9461-45e2-ad09-a1b0259ff68e"
-					(reference "Q18")
+					(reference "Q19")
 					(unit 1)
 				)
@@
 		(dnp no)
 		(fields_autoplaced yes)
-		(property "Reference" "Q6"
+		(property "Reference" "Q7"
 			(at 46.99 115.5699 0)
 			(effects
@@
 			(project "Omega Radio"
 				(path "/3468ce30-82a7-4087-a7ac-02063723d842/ec53c5ee-9461-45e2-ad09-a1b0259ff68e"
-					(reference "Q6")
+					(reference "Q7")
 					(unit 1)
 				)
@@
 		(on_board yes)
 		(dnp no)
-		(property "Reference" "Q9"
+		(property "Reference" "Q10"
 			(at 94.488 36.83 0)
 			(effects
@@
 			(project ""
 				(path "/3468ce30-82a7-4087-a7ac-02063723d842/ec53c5ee-9461-45e2-ad09-a1b0259ff68e"
-					(reference "Q9")
+					(reference "Q10")
 					(unit 1)
 				)
@@
 		(on_board yes)
 		(dnp no)
-		(property "Reference" "Q15"
+		(property "Reference" "Q16"
 			(at 182.626 52.578 0)
 			(effects
@@
 			(project "Omega Radio"
 				(path "/3468ce30-82a7-4087-a7ac-02063723d842/ec53c5ee-9461-45e2-ad09-a1b0259ff68e"
-					(reference "Q15")
+					(reference "Q16")
 					(unit 1)
 				)
@@
 		(dnp no)
 		(fields_autoplaced yes)
-		(property "Reference" "Q13"
+		(property "Reference" "Q14"
 			(at 135.89 92.7099 0)
 			(effects
@@
 			(project "Omega Radio"
 				(path "/3468ce30-82a7-4087-a7ac-02063723d842/ec53c5ee-9461-45e2-ad09-a1b0259ff68e"
-					(reference "Q13")
+					(reference "Q14")
 					(unit 1)
 				)

Commit message: AGC Work 4
Parts:
- renumbered C96 to C100, C97 to C101, C98 to C102, C99 to C103, C100 to C104, C53 to C57, C54 to C58, C55 to C59, C56 to C60, C57 to C61, C58 to C62, C59 to C63, C60 to C64, C61 to C65, C62 to C66, C63 to C67, C64 to C68, C65 to C69, C66 to C70, C67 to C71, C68 to C72, C69 to C73, C70 to C74, C71 to C75, C72 to C76, C73 to C77, C74 to C78, C75 to C79, C76 to C80, C77 to C81, C78 to C82, C79 to C83, C80 to C84, C81 to C85, C82 to C86, C83 to C87, C84 to C88, C85 to C89, C86 to C90, C87 to C91, C88 to C92, C89 to C93, C90 to C94, C91 to C95, C92 to C96, C93 to C97, C94 to C98, C95 to C99, R44 to R49, R45 to R50, R46 to R51, R47 to R52, R48 to R53, R49 to R54, R50 to R55, R51 to R56

Commit message: All AGCs done
Parts:
- renumbered C98 to C100, C99 to C101, C100 to C102, C101 to C103, C102 to C104, C103 to C105, C104 to C106, C57 to C59, C58 to C60, C59 to C61, C60 to C62, C61 to C63, C62 to C64, C63 to C65, C64 to C66, C65 to C67, C66 to C68, C67 to C69, C68 to C70, C69 to C71, C70 to C72, C71 to C73, C72 to C74, C73 to C75, C74 to C76, C75 to C77, C76 to C78, C77 to C79, C78 to C80, C79 to C81, C80 to C82, C81 to C83, C82 to C84, C83 to C85, C84 to C86, C85 to C87, C86 to C88, C87 to C89, C88 to C90, C89 to C91, C90 to C92, C91 to C93, C92 to C94, C93 to C95, C94 to C96, C95 to C97, C96 to C98, C97 to C99, R49 to R57, R50 to R58, R51 to R59, R52 to R60, R53 to R61, R54 to R62, R55 to R63, R56 to R64
