File: LPF(PA cont).kicad_sch (KiCad schematic)
At the start: 28 parts, among them K1 G5V-1, K2 G5V-1, K3 G5V-1, K4 G5V-1, K5 G5V-1, K6 G5V-1, K7 G5V-1, K8 G5V-1

Commit message: All AGCs done
Parts:
- renumbered C154 to C156, C155 to C157, C156 to C158, C157 to C159, C158 to C160, C159 to C161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
